Commit message: 实现初步闭环

File: src/cchess_ros_control/machinery_chess_bringup/urdf/machinery.urdf.xacro (robot description, xacro)
@@ -3,4 +3,5 @@
     <!-- 参数 -->
     <xacro:arg name="origin_position" default="[180.0, 0.0, 444.2]"/>
+    <xacro:arg name="custom_origin_position" default="[180.0, 0.0, 444.2]"/>
     <xacro:arg name="frame_prefix" default=""/>
     <xacro:arg name="serial_port_name" default="/dev/ttyUSB0" />
@@ -12,4 +13,4 @@
     <!-- 2. 调用宏并传入 frame_prefix 参数 -->
     <xacro:machinery_model frame_prefix="$(arg frame_prefix)"/>
-    <xacro:machinery_control origin_position="$(arg origin_position)" frame_prefix="$(arg frame_prefix)" serial_port_name="$(arg serial_port_name)" />
+    <xacro:machinery_control origin_position="$(arg origin_position)" custom_origin_position="$(arg custom_origin_position)" frame_prefix="$(arg frame_prefix)" serial_port_name="$(arg serial_port_name)" />
 </robot>

File: src/cchess_ros_control/machinery_chess_bringup/urdf/machinery_control.urdf.xacro (robot description, xacro)
@@ -1,14 +1,17 @@
 <?xml version="1.0" encoding="utf-8"?>
 <robot name="Machinery" xmlns:xacro="http://www.ros.org/wiki/xacro">
-  <xacro:macro name="machinery_control" params="origin_position frame_prefix serial_port_name">
+  <xacro:macro name="machinery_control" params="origin_position custom_origin_position frame_prefix serial_port_name">
     <ros2_control name="MachineryRobotSystem" type="system">
+      <!-- 指定 hardware_interface 插件 -->
       <hardware>
         <plugin>machinery_hardware_interface/MachineryHardwareInterface</plugin>
         <param name="origin_position">$(arg origin_position)</param>
+        <param name="custom_origin_position">$(arg custom_origin_position)</param>
         <param name="frame_prefix">$(arg frame_prefix)</param>
         <param name="serial_port_name">$(arg serial_port_name)</param>
 <!--        <param name="baud_rate">$(arg baud_rate)</param>-->
       </hardware>
-      <joint name="${frame_prefix}joint5">
+      <!-- 声明 hardware_interface的接口 -->
+      <joint name="$(arg frame_prefix)gripper_position">
         <command_interface name="x_position"/>
         <command_interface name="y_position"/>
@@ -18,7 +21,7 @@
         <state_interface name="z_position"/>
       </joint>
-      <joint name="${frame_prefix}gripper_joint">
-        <command_interface name="enable"/>
-        <state_interface name="enable"/>
+      <joint name="$(arg frame_prefix)gripper_suction">
+        <command_interface name="position"/>
+        <state_interface name="position"/>
       </joint>
     </ros2_control>

File: src/cchess_ros_control/machinery_ros2control/machinery_ros2control_bringup/urdf/machinery_control.urdf.xacro (robot description, xacro)
@@ -1,14 +1,15 @@
 <?xml version="1.0" encoding="utf-8"?>
 <robot name="Machinery" xmlns:xacro="http://www.ros.org/wiki/xacro">
-  <xacro:macro name="machinery_control" params="origin_position frame_prefix serial_port_name">
+  <xacro:macro name="machinery_control" params="origin_position custom_origin_position frame_prefix serial_port_name">
     <ros2_control name="MachineryRobotSystem" type="system">
       <hardware>
         <plugin>machinery_hardware_interface/MachineryHardwareInterface</plugin>
         <param name="origin_position">$(arg origin_position)</param>
+        <param name="custom_origin_position">$(arg custom_origin_position)</param>
         <param name="frame_prefix">$(arg frame_prefix)</param>
         <param name="serial_port_name">$(arg serial_port_name)</param>
 <!--        <param name="baud_rate">$(arg baud_rate)</param>-->
       </hardware>
-      <joint name="$(arg frame_prefix)joint5">
+      <joint name="$(arg frame_prefix)gripper_position">
         <command_interface name="x_position"/>
         <command_interface name="y_position"/>
@@ -18,7 +19,7 @@
         <state_interface name="z_position"/>
       </joint>
-      <joint name="$(arg frame_prefix)gripper_joint">
-        <command_interface name="enable"/>
-        <state_interface name="enable"/>
+      <joint name="$(arg frame_prefix)gripper_suction">
+        <command_interface name="position"/>
+        <state_interface name="position"/>
       </joint>
     </ros2_control>
